File: AV_MOD_FAMICOM.kicad_sch (KiCad schematic)
At the start: 13 parts, among them J1 USB-A-S-X-X-TH, J2 USB-A-S-X-X-TH, J3 Conn_01x02_Male, J5 Conn_01x07, Q1 Q_PNP_CBE, Q2 Q_NPN_CBE

Commit message: Add files via upload
New version of the board
Parts:
- removed D1: DIODE, Diode_THT:D_5W_P12.70mm_Horizontal, symbol pspice:DIODE
- removed Q2: Q_NPN_CBE, Package_TO_SOT_THT:TO-92, symbol Device:Q_NPN_CBE
- removed R3: 68, Resistor_THT:R_Axial_DIN0207_L6.3mm_D2.5mm_P10.16mm_Horizontal, symbol Device:R
- removed R4: 82?, Resistor_THT:R_Axial_DIN0207_L6.3mm_D2.5mm_P10.16mm_Horizontal, symbol Device:R
- J1: footprint SAMTEC_USB-A-S-X-X-TH -> USB-A-S-X-X-TH:SAMTEC_USB-A-S-X-X-TH
- J2: footprint SAMTEC_USB-A-S-X-X-TH -> USB-A-S-X-X-TH:SAMTEC_USB-A-S-X-X-TH; FARNELL (none) -> https://fr.farnell.com/samtec/usb-a-s-f-b-th/conn-usb-2-0-t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
- R1: value 2200 -> 150
- R2: value 220 -> 100
Connections:
- net GNDREF: now also J1.S1 (SHIELD), J1.S2 (SHIELD), J2.S1 (SHIELD), J2.S2 (SHIELD)
- net VIDEO OUT: now also C1.2
- net at R1.2, R2.1: now also C1.1
Other:
- moved on the sheet: C1
